Commit message: Add Docker setup and desk cleaning support

File: src/armpi_fpv_descrption/urdf/armpi_fpv.urdf (robot description, URDF)
Before this commit: robot armpi_fpv_description, 16 links, 15 joints
Joints:
- joint r_joint: limit lower=-1.57 upper=1.57 effort=1000 velocity=5 -> lower=-2.10 upper=1.26 effort=1000 velocity=5
